File: KiCad/BLDCControl1.kicad_Lolin32Lite_sch.kicad_sch (KiCad schematic)
At the start: 40 parts, among them J2 Conn_Power, J3 Conn BLDC, Q1 IRLZ44N, Q2 IRLZ44N, Q3 IRLZ44N, Q4 IRLZ44N, Q5 IRLZ44N, Q6 IRLZ44N, U1 IR2101, U2 IR2101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

Commit message: kicad update
Parts:
- removed U4: ~, symbol WemosLolin32Lite:WemosLolin32Lite_DIP26
- added C6, C7, C8: 220uF, Capacitor_THT:CP_Radial_D6.3mm_P2.50mm, symbol Device:C_Polarized
- added R16: 10k, Resistor_THT:R_Axial_DIN0204_L3.6mm_D1.6mm_P5.08mm_Horizontal, symbol Device:R
- added U10: STM32F411CE_BlackPill, Package_DIP:DIP-40_W15.24mm, symbol New_Library:STM32F411CE_BlackPill
- added WemosLolin32Lite1: ~, lolin32-lite-1.snapshot.18:DIP-26_900_WEMOS_LOLIN32_LITE, symbol WemosLolin32Lite:Wemos{colon}_DIP26
- U6: footprint (none) -> Package_DIP:DIP-14_W7.62mm
- U7, U8, U9: footprint (none) -> Package_DIP:CERDIP-14_W7.62mm_SideBrazed
Connections:
- net +15V: now also C6.1, C7.1, C8.1
- net +5V: now also U7.14 (VDD), U8.14 (VDD), U9.14 (VCC), R16.1, U10.18 (5V)
- net EMF_AC: now also U10.28 (PA2), WemosLolin32Lite1.18 (GPIO4)
- net EMF_BA: now also U10.27 (PA1), WemosLolin32Lite1.19 (GPIO16)
- net EMF_CB: now also U10.26 (PA0), WemosLolin32Lite1.20 (GPIO17)
- net GND: now also U7.7 (VSS), U8.7 (VSS), U9.7 (GND), C6.2, C7.2, C8.2, U10.19 (VSS), U10.35 (PB1), U10.47 (VSS), U10.49 (VSS), WemosLolin32Lite1.13 (GND)
- net PWM_AH: now also U9.2, U10.1 (PB12); no longer U9.12
- net PWM_AL: now also U9.12, U10.2 (PB13); no longer U9.10
- net PWM_BH: now also U9.4, U10.3 (PB14); no longer U9.8
- net PWM_BL: now also U9.10, U10.4 (PB15); no longer U9.6
- net PWM_CH: now also U9.6, U10.16 (PB8); no longer U9.4
- net SCL: now also WemosLolin32Lite1.24 (GPIO19)
- net SDA: now also WemosLolin32Lite1.22 (GPIO18)
- net at U9.11: now also U8.3; no longer U8.10
- net at U9.9: now also U7.11; no longer U8.4
- net at U9.5: now also U7.3; no longer U8.3
- net at U8.11: now also U9.1; no longer U9.13
- net at U8.12: now also WemosLolin32Lite1.6 (GPIO32)
- net at U7.13, U7.4, U8.13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: now also U7.2; no longer U7.9
- net at U9.3: now also U8.4; no longer U7.11
- net at U7.12: now also WemosLolin32Lite1.11 (GPIO14)
- net at U8.8: now also WemosLolin32Lite1.7 (GPIO33)
- net at U8.5: now also WemosLolin32Lite1.8 (GPIO25)
- net at U7.10: now also U7.5, U7.6; no longer U9.1
- net at U7.8: now also WemosLolin32Lite1.12 (GPIO12)
- net at U7.1: now also WemosLolin32Lite1.10 (GPIO27); no longer U7.2
- net at U8.1: now also WemosLolin32Lite1.9 (GPIO26)
- net EMF_COMMON: no longer names the net of R13.1, R14.1, R15.1
- net PWM_LH renamed PWM_CL
- net PWM_CL: now also U9.8, U10.17 (PB9); no longer U9.2
- new net: U8.10, U9.13
- new net: R16.2, U7.9
Other:
- moved on the sheet: U7A, U7C, U7D, U7E, U8E, U9A, U9B, U9C, U9D, U9E, U9F, U9G

Commit message: Lolin32 bldc
Parts:
- removed R16: 10k, Resistor_THT:R_Axial_DIN0204_L3.6mm_D1.6mm_P5.08mm_Horizontal, symbol Device:R
Connections:
- net PWM_AH: now also U9.10; no longer U9.2
- net PWM_BL: now also U9.2; no longer U9.10
- net at WemosLolin32Lite1.10 (GPIO27): now also U7.12; no longer U7.1
- net at WemosLolin32Lite1.11 (GPIO14): now also U7.1; no longer U7.12
- net at WemosLolin32Lite1.12 (GPIO12): now also U7.5, U7.6; no longer U7.8
- net at WemosLolin32Lite1.6 (GPIO32): now also U8.1; no longer U8.12
- net at WemosLolin32Lite1.7 (GPIO33): now also U8.13; no longer U8.8
- net at WemosLolin32Lite1.8 (GPIO25): now also U8.6; no longer U8.5
- net at WemosLolin32Lite1.9 (GPIO26): now also U8.9; no longer U8.1
- net at U9.11: now also U7.3; no longer U8.3
- net at U9.5: now also U8.10; no longer U7.3
- net at U9.13: now also U8.4; no longer U8.10
- net at U9.3: now also U8.3; no longer U8.4
- net at U7.9: now also U7.4, U7.8
- new net: U7.10, U7.13, U7.2, U8.12, U8.2, U8.5, U8.8
Other:
- moved on the sheet: U9B, U9C, U9E, U9F

Commit message: current measure kicad
Parts:
- removed J3: Conn BLDC, Connector_PinSocket_2.54mm:PinSocket_1x03_P2.54mm_Vertical, symbol Connector:Conn_01x03_Socket
- removed R11, R12: 10k, Resistor_THT:R_Axial_DIN0204_L3.6mm_D1.6mm_P5.08mm_Horizontal, symbol Device:R
- removed R13, R14, R15: 47k, Resistor_THT:R_Axial_DIN0204_L3.6mm_D1.6mm_P5.08mm_Horizontal, symbol Device:R
- removed U6: LM339, Package_DIP:DIP-14_W7.62mm, symbol Comparator:LM339
- removed unit 7 of U9
- added U4: LM393, symbol Comparator:LM393
- R10: footprint Resistor_THT:R_Axial_DIN0204_L3.6mm_D1.6mm_P5.08mm_Horizontal -> (none)
- R7, R8: value 47k -> 20m; footprint Resistor_THT:R_Axial_DIN0204_L3.6mm_D1.6mm_P5.08mm_Horizontal -> (none)
- R9: value 47k -> 10k; footprint Resistor_THT:R_Axial_DIN0204_L3.6mm_D1.6mm_P5.08mm_Horizontal -> (none)
Connections:
- net +15V: now also U4.8 (V+)
- net BLDC_A: now also U4.2 (-)
- net BLDC_B: now also U4.6 (-)
- net BLDC_C: no longer R9.2
- net GND: now also U4.4 (V-); no longer R10.2
- net +3.3V: now reaches R10.1
- net +3.3V: now also R9.1; no longer R7.1
- net BLDC_BP: now reaches R8.1
- net BLDC_BP: now also U4.5 (+)
- new net BLDC_AP: R7.1, U4.3 (+)
- new net EMF_A: R9.2, U4.1
- new net EMF_B: R10.2, U4.7
